Commit message: modify file schema

File: mybot_description/diffbot_description/urdf/diffbot_base.urdf.xacro (robot description, xacro)
@@ -19,5 +19,5 @@
     <xacro:property name="base_link_radius" value="0.205" /> <!-- base_link 半径 -->
     <xacro:property name="base_link_height" value="0.2" /> <!-- base_link 长 -->
-    <xacro:property name="earth_space" value="0.14" /> <!-- 离地间距 -->
+    <xacro:property name="earth_space" value="0.04" /> <!-- 离地间距 -->
     <xacro:property name="base_link_m" value="5" /> <!-- 质量  -->
     <!-- 底盘 -->
@@ -81,18 +81,7 @@
         <parent link="base_link" />
         <child link="${name}_wheel" />
-        <origin xyz="0 ${flag * (base_link_radius - wheel_length / 2)} ${-(earth_space + base_link_height / 2 - wheel_radius) }" />
+        <origin xyz="0 ${flag * (base_link_radius - wheel_length / 2)} ${-(earth_space + base_link_height / 2 - wheel_radius) - 0.0001 }" />
         <axis xyz="0 1 0" />
       </joint>
-        <!-- Transmission is important to link the joints and the controller -->
-      <transmission name="${name}_wheel2base_link_trans">
-          <type>transmission_interface/SimpleTransmission</type>
-          <joint name="${name}_wheel2base_link">
-                <hardwareInterface>hardware_interface/VelocityJointInterface</hardwareInterface>
-          </joint>
-          <actuator name="${name}_wheel2base_link_motor">
-                <hardwareInterface>hardware_interface/VelocityJointInterface</hardwareInterface>
-                <mechanicalReduction>30</mechanicalReduction>
-          </actuator>
-      </transmission>
       <gazebo reference="${name}_wheel">
         <material>Gazebo/Red</material>
@@ -103,5 +92,5 @@
     <!-- 支撑轮 -->
     <!-- 支撑轮属性 -->
-    <xacro:property name="support_wheel_radius" value="0.07" /> <!-- 支撑轮半径 -->
+    <xacro:property name="support_wheel_radius" value="0.02" /> <!-- 支撑轮半径 -->
     <xacro:property name="support_wheel_m" value="0.3" /> <!-- 质量  -->
     <!-- 支撑轮宏 -->

File: mybot_description/diffbot_description/urdf/diffbot_sim.urdf.xacro (robot description, xacro)
@@ -4,5 +4,3 @@
     <xacro:include filename="$(find mybot_description)/diffbot_description/urdf/diffbot.urdf.xacro" />
     <xacro:include filename="$(find mybot_description)/diffbot_description/urdf/plugin/gazebo_ros_control.urdf.xacro" />
-    <!-- <xacro:include filename="$(find mybot_description)/model/sensor/sensors_laser.urdf.xacro" /> -->
-    <!-- <xacro:include filename="$(find mybot_description)/model/sensor/sensors_camera.urdf.xacro" /> -->
 </robot>

File: mybot_description/diffbot_description/urdf/diffbot_sim_gazebo_control.urdf.xacro (robot description, xacro)
@@ -4,5 +4,3 @@
     <xacro:include filename="$(find mybot_description)/diffbot_description/urdf/diffbot.urdf.xacro" />
     <xacro:include filename="$(find mybot_description)/diffbot_description/urdf/plugin/gazebo_diff_drive.urdf.xacro" />
-    <!-- <xacro:include filename="$(find mybot_description)/model/sensor/sensors_laser.urdf.xacro" /> -->
-    <!-- <xacro:include filename="$(find mybot_description)/model/sensor/sensors_camera.urdf.xacro" /> -->
 </robot>

File: mybot_description/diffbot_description/urdf/plugin/gazebo_diff_drive.urdf.xacro (robot description, xacro)
@@ -13,5 +13,5 @@
             <leftJoint>left_wheel2base_link</leftJoint> <!-- 左轮 -->
             <rightJoint>right_wheel2base_link</rightJoint> <!-- 右轮 -->
-            <wheelSeparation>${base_link_radius * 2}</wheelSeparation> <!-- 车轮间距 -->
+            <wheelSeparation>${base_link_radius * 2 - wheel_length }</wheelSeparation> <!-- 车轮间距 -->
             <wheelDiameter>${wheel_radius * 2}</wheelDiameter> <!-- 车轮直径 -->
             <broadcastTF>1</broadcastTF>

File: mybot_description/diffbot_description/urdf/plugin/gazebo_ros_control.urdf.xacro (robot description, xacro)
@@ -1,3 +1,18 @@
 <robot name="gazebo_ros_control" xmlns:xacro="http://wiki.ros.org/xacro">
+	<xacro:macro name="add_wheels_transmission" params="name">
+		<!-- Transmission is important to link the joints and the controller -->
+		<transmission name="${name}_wheel2base_link_trans">
+			<type>transmission_interface/SimpleTransmission</type>
+			<joint name="${name}_wheel2base_link">
+				<hardwareInterface>hardware_interface/VelocityJointInterface</hardwareInterface>
+			</joint>
+			<actuator name="${name}_wheel2base_link_motor">
+				<hardwareInterface>hardware_interface/VelocityJointInterface</hardwareInterface>
+				<mechanicalReduction>1</mechanicalReduction>
+			</actuator>
+		</transmission>
+	</xacro:macro>
+	<xacro:add_wheels_transmission name="left" />
+	<xacro:add_wheels_transmission name="right" />
 	<!-- ros_control plugin -->
 	<gazebo>

File: mybot_description/mecanumbot_description/urdf/mecanumbot_base.urdf.xacro (robot description, xacro)
@@ -87,14 +87,4 @@
         <axis xyz="0 1 0" />
       </joint>
-        <!-- Transmission is important to link the joints and the controller -->
-      <transmission name="${name}_wheel2base_link_trans">
-          <type>transmission_interface/SimpleTransmission</type>
-          <joint name="${name}_wheel2base_link">
-                <hardwareInterface>hardware_interface/EffortJointInterface</hardwareInterface>
-          </joint>
-          <actuator name="${name}_wheel2base_link_motor">
-                <mechanicalReduction>1</mechanicalReduction>
-          </actuator>
-      </transmission>
       <gazebo reference="${name}_wheel">
         <material>Gazebo/Red</material>

File: mybot_description/mecanumbot_description/urdf/plugin/gazebo_ros_control.urdf.xacro (robot description, xacro)
@@ -1,3 +1,23 @@
 <robot name="gazebo_ros_control" xmlns:xacro="http://wiki.ros.org/xacro">
+	<!-- Transmission is important to link the joints and the controller -->
+	<xacro:macro name="add_wheels_transmission" params="name">
+		<transmission name="${name}_wheel2base_link_trans">
+			<type>transmission_interface/SimpleTransmission</type>
+			<joint name="${name}_wheel2base_link">
+				<hardwareInterface>hardware_interface/VelocityJointInterface</hardwareInterface>
+			</joint>
+			<actuator name="${name}_wheel2base_link_motor">
+				<hardwareInterface>hardware_interface/VelocityJointInterface</hardwareInterface>
+				<mechanicalReduction>1</mechanicalReduction>
+			</actuator>
+		</transmission>
+		<gazebo reference="${name}_wheel">
+			<material>Gazebo/Red</material>
+		</gazebo>
+	</xacro:macro>
+	<xacro:add_wheels_transmission name="left_front"/>
+	<xacro:add_wheels_transmission name="right_front"/>
+	<xacro:add_wheels_transmission name="left_rear"/>
+	<xacro:add_wheels_transmission name="right_rear"/>
 	<!-- ros_control plugin -->
 	<gazebo>
